Commit message: trash commit just to checkout hash

File: install/simple_robot_description/share/simple_robot_description/urdf/simple_robot.xacro (robot description, xacro)
@@ -1,208 +1 @@
-<?xml version="1.0"?>
-<robot xmlns:xacro="http://www.ros.org/wiki/xacro" name="simple_robot">
-  <!-- Base Link -->
-  <link name="base_link">
-    <visual>
-      <geometry>
-        <box size="0.5 0.3 0.1"/>
-      </geometry>
-      <material name="blue">
-        <color rgba="0 0 1 1"/>
-      </material>
-    </visual>
-    <collision>
-      <geometry>
-        <box size="0.5 0.3 0.1"/>
-      </geometry>
-    </collision>
-    <inertial>
-      <mass value="5.0"/>
-      <origin xyz="0 0 0" rpy="0 0 0"/>
-      <inertia ixx="0.1" ixy="0.0" ixz="0.0" iyy="0.1" iyz="0.0" izz="0.1"/>
-    </inertial>
-  </link>
-  <!-- Wheels -->
-  <xacro:macro name="wheel" params="name x y z">
-    <link name="${name}">
-      <visual>
-        <geometry>
-          <cylinder length="0.05" radius="0.1"/>
-        </geometry>
-        <origin rpy="1.5708 0 0"/>
-        <material name="black">
-          <color rgba="0 0 0 1"/>
-        </material>
-      </visual>
-      <collision>
-        <geometry>
-          <cylinder length="0.05" radius="0.1"/>
-        </geometry>
-        <origin rpy="1.5708 0 0"/>
-      </collision>
-      <inertial>
-        <mass value="1.0"/>
-        <origin xyz="0 0 0" rpy="0 0 0"/>
-        <inertia ixx="0.01" ixy="0.0" ixz="0.0" iyy="0.01" iyz="0.0" izz="0.01"/>
-      </inertial>
-    </link>
-    <joint name="${name}_joint" type="continuous">
-      <parent link="base_link"/>
-      <child link="${name}"/>
-      <origin xyz="${x} ${y} ${z}" rpy="0 0 0"/>
-      <axis xyz="0 1 0"/>
-    </joint>
-  </xacro:macro>
-  <xacro:wheel name="front_left_wheel" x="0.2" y="0.2" z="0.0"/>
-  <xacro:wheel name="front_right_wheel" x="0.2" y="-0.2" z="0.0"/>
-  <xacro:wheel name="rear_right_wheel" x="-0.2" y="-0.2" z="0.0"/>
-  <!-- <xacro:wheel name="rear_left_wheel" x="-0.2" y="0.2" z="0.0"/> -->
-  <!-- REAR LEFT WHEEL (ЯВНО) -->
-  <link name="rear_left_wheel">
-    <visual>
-      <geometry>
-        <cylinder length="0.05" radius="0.1"/>
-      </geometry>
-      <origin rpy="1.5708 0 0"/>
-      <material name="black">
-        <color rgba="0 0 0 1"/>
-      </material>
-    </visual>
-    <collision>
-      <geometry>
-        <cylinder length="0.05" radius="0.1"/>
-      </geometry>
-      <origin rpy="1.5708 0 0"/>
-    </collision>
-    <inertial>
-      <mass value="1.0"/>
-      <origin xyz="0 0 0" rpy="0 0 0"/>
-      <inertia ixx="0.01" ixy="0.0" ixz="0.0" iyy="0.01" iyz="0.0" izz="0.01"/>
-    </inertial>
-  </link>
-  <joint name="rear_left_wheel_joint" type="continuous">
-    <parent link="base_link"/>
-    <child link="rear_left_wheel"/>
-    <origin xyz="-0.2 0.2 0.0" rpy="0 0 0"/>
-    <axis xyz="0 -1 0"/>
-  </joint>
-  <!-- Camera -->
-  <link name="camera_link">
-    <visual>
-      <geometry>
-        <box size="0.1 0.1 0.1"/>
-      </geometry>
-      <material name="gray">
-        <color rgba="0.5 0.5 0.5 1"/>
-      </material>
-    </visual>
-  </link>
-  <joint name="camera_joint" type="fixed">
-    <parent link="base_link"/>
-    <child link="camera_link"/>
-    <origin xyz="0.2 0 0.1" rpy="0 0 0"/>
-  </joint>
-  <gazebo reference="camera_link">
-  <sensor type="camera" name="camera_sensor">
-    <always_on>true</always_on>
-    <visualize>true</visualize>
-    <update_rate>30.0</update_rate>
-    <camera>
-      <horizontal_fov>1.3962634</horizontal_fov>
-      <image>
-        <width>640</width>
-        <height>480</height>
-        <format>R8G8B8</format>
-      </image>
-      <clip>
-        <near>0.1</near>
-        <far>100.0</far>
-      </clip>
-    </camera>
-    <plugin name="gazebo_ros_camera" filename="libgazebo_ros_camera.so">
-      <robotNamespace>/</robotNamespace>
-      <cameraName>camera</cameraName>
-      <imageTopicName>camera/image_raw</imageTopicName>
-      <cameraInfoTopicName>camera/camera_info</cameraInfoTopicName>
-      <frameName>camera_link</frameName>
-      <qos_camera>best_effort</qos_camera>
-    </plugin>
-  </sensor>
-</gazebo>
-  <!-- Lidar -->
-  <link name="lidar_link">
-    <visual>
-      <geometry>
-        <cylinder length="0.1" radius="0.05"/>
-      </geometry>
-      <material name="red">
-        <color rgba="1 0 0 1"/>
-      </material>
-    </visual>
-  </link>
-  <joint name="lidar_joint" type="fixed">
-    <parent link="base_link"/>
-    <child link="lidar_link"/>
-    <origin xyz="0.1 0 0.15" rpy="0 0 0"/>
-  </joint>
-  <gazebo reference="lidar_link">
-    <sensor name="lidar_sensor" type="ray">
-      <ray>
-        <scan>
-          <horizontal>
-            <samples>720</samples>
-            <resolution>1</resolution>
-            <min_angle>-1.57</min_angle>
-            <max_angle>1.57</max_angle>
-          </horizontal>
-        </scan>
-        <range>
-          <min>0.1</min>
-          <max>10.0</max>
-          <resolution>0.01</resolution>
-        </range>
-      </ray>
-      <always_on>true</always_on>
-      <update_rate>30</update_rate>
-      <visualize>true</visualize>
-    </sensor>
-    <plugin name="gazebo_ros_ray_sensor" filename="libgazebo_ros_ray_sensor.so">
-      <ros>
-        <namespace>/</namespace>
-        <remapping>scan:=scan</remapping>
-      </ros>
-      <frame_name>lidar_link</frame_name>
-    </plugin>
-  </gazebo>
-  <gazebo reference="front_left_wheel">
-    <mu1>0.0</mu1>
-    <mu2>0.0</mu2>
-    <dampingFactor>0.0</dampingFactor>
-    <fdir1>0 0 0</fdir1>
-    <gravity>false</gravity>
-  </gazebo>
-  <gazebo reference="front_right_wheel">
-    <mu1>0.0</mu1>
-    <mu2>0.0</mu2>
-    <dampingFactor>0.0</dampingFactor>
-    <fdir1>0 0 0</fdir1>
-    <gravity>false</gravity>
-  </gazebo>
-  <!-- Diff Drive Plugin -->
-  <gazebo>
-    <plugin name="diff_drive_controller" filename="libgazebo_ros_diff_drive.so">
-      <ros>
-        <namespace>/</namespace>
-        <remapping>cmd_vel:=/cmd_vel</remapping>
-        <remapping>odom:=/odom</remapping>
-      </ros>
-      <update_rate>30</update_rate>
-      <left_joint>rear_left_wheel_joint</left_joint>
-      <right_joint>rear_right_wheel_joint</right_joint>
-      <wheel_separation>0.4</wheel_separation>
-      <wheel_diameter>0.2</wheel_diameter>
-      <publish_odom>true</publish_odom>
-      <odometry_frame>odom</odometry_frame>
-      <robot_base_frame>base_link</robot_base_frame>
-    </plugin>
-  </gazebo>
-</robot>
+/home/elisey/ros2_ws/src/simple_robot_description/urdf/simple_robot.xacro

Commit message: fixed camerain xacro, deleted slam toolbox, setup rtab

File: install/simple_robot_description/share/simple_robot_description/urdf/simple_robot.xacro (robot description, xacro)
@@ -88,42 +88,45 @@
   <!-- Camera -->
   <link name="camera_link">
-    <visual>
-      <geometry>
-        <box size="0.1 0.1 0.1"/>
-      </geometry>
-      <material name="gray">
-        <color rgba="0.5 0.5 0.5 1"/>
-      </material>
-    </visual>
-  </link>
-  <joint name="camera_joint" type="fixed">
-    <parent link="base_link"/>
-    <child link="camera_link"/>
-    <origin xyz="0.2 0 0.1" rpy="0 0 0"/>
-  </joint>
-  <gazebo reference="camera_link">
-    <sensor type="camera" name="camera_sensor">
-      <update_rate>30.0</update_rate>
-      <camera>
-        <horizontal_fov>1.3962634</horizontal_fov>
-        <image>
-          <width>640</width>
-          <height>480</height>
-          <format>R8G8B8</format>
-        </image>
-        <clip>
-          <near>0.1</near>
-          <far>100.0</far>
-        </clip>
-      </camera>
-      <plugin name="gazebo_ros_camera" filename="libgazebo_ros_camera.so">
-        <robotNamespace>/</robotNamespace>
-        <cameraName>camera</cameraName>
-        <imageTopicName>camera/image_raw</imageTopicName>
-        <cameraInfoTopicName>camera/camera_info</cameraInfoTopicName>
-        <frameName>camera_link</frameName>
-      </plugin>
-    </sensor>
-  </gazebo>
+     <visual>
+       <geometry>
+         <box size="0.1 0.1 0.1"/>
+       </geometry>
+       <material name="gray">
+         <color rgba="0.5 0.5 0.5 1"/>
+       </material>
+     </visual>
+   </link>
+   <joint name="camera_joint" type="fixed">
+     <parent link="base_link"/>
+     <child link="camera_link"/>
+     <origin xyz="0.2 0 0.1" rpy="0 0 0"/>
+   </joint>
+   <gazebo reference="camera_link">
+     <sensor type="camera" name="camera_sensor">
+     <always_on>true</always_on>
+     <visualize>true</visualize>
+     <update_rate>30.0</update_rate>
+     <camera>
+       <horizontal_fov>1.3962634</horizontal_fov>
+       <image>
+         <width>640</width>
+         <height>480</height>
+         <format>R8G8B8</format>
+       </image>
+       <clip>
+         <near>0.1</near>
+         <far>100.0</far>
+       </clip>
+     </camera>
+     <plugin name="gazebo_ros_camera" filename="libgazebo_ros_camera.so">
+       <robotNamespace>/</robotNamespace>
+       <cameraName>camera</cameraName>
+       <imageTopicName>camera/image_raw</imageTopicName>
+       <cameraInfoTopicName>camera/camera_info</cameraInfoTopicName>
+       <frameName>camera_link</frameName>
+       <qos_camera>best_effort</qos_camera>
+     </plugin>
+   </sensor>
+   </gazebo>
   <!-- Lidar -->
   <link name="lidar_link">
